File: ArduinoMiniPro Breakout.brd (EAGLE design)
At the start: 266.7 x 48.3 mm, 58 parts, among them IC1 4050N, IC2 4050N, IC3 74HC00N, IC4 74HC00N, IC5 74HC00N, IC6 74HC00N, IC7 74HC00N, IC8 74HC00N, IC9 74HC00N

Commit message: Made the board a pure breakout board
Rather than smooshing all the functions onto a single board, this board
is purely for breaking out the pins to headers.

Given the relatively large size, there is no reason a full size Arduino
cannot be used, and so a full size breakout is on the way.
Parts:
- removed C2, C3, C4, C5: 10uF, SparkFun-Capacitors:CPOL-RADIAL-10UF-25V
- removed IC1, IC2: 4050N, 40xx:DIL16
- removed IC3, IC4, IC5, IC6, IC7, IC8, IC9: 74HC00N, 74xx-eu:DIL14
- removed JP10, JP11, JP12, JP13, JP14, JP15, JP16, JP17, JP7, JP9: (no value), MY-Connectors:SCREWTERMINAL-5MM-3
- removed LED1, LED2, LED3, LED4, LED5, LED6, LED7: (no value), SparkFun-LED:LED3MM
- removed R13, R14, R15, R16: 10k0, resistor:0207/7
- removed R17, R18, R19, R24, R25, R26, R27: 150, resistor:0207/7
- removed R20, R21, R22, R23: 1k00, resistor:0207/10
- removed RN1, RN2: 680, resistor-dil:DIL16
- added C1: 47uF, SparkFun-Passives:CPOL-RADIAL-10UF-25V
- added SV1, SV11, SV4: (no value), con-lstb:MA03-1
- added SV10, SV9: (no value), SparkFun-Connectors:SCREWTERMINAL-5MM-3
- added SV6: (no value), con-lstb:MA04-1
- JP1, JP2, JP3, JP4, JP5, JP6: device MY-Connectors:SCREWTERMINAL-5MM-3 -> SparkFun-Connectors:SCREWTERMINAL-5MM-3
- moved JP1 229.2 mm to (5.08, 104.1), turned to 270 degrees
- moved JP2 210.8 mm to (5.08, 88.9), turned to 270 degrees
- moved JP3 192.9 mm to (5.08, 73.7), turned to 270 degrees
- moved U$2 183.2 mm to (43.2, 66.0), turned to 0 degrees
- moved JP4 175.9 mm to (5.08, 58.4), turned to 270 degrees
- moved JP0 169.5 mm to (96.5, 99.1), turned to 90 degrees
- moved JP5 160.0 mm to (5.08, 43.2), turned to 270 degrees
- moved JP6 145.6 mm to (5.08, 27.9), turned to 270 degrees
- moved SV2 113.4 mm to (96.5, 48.3), turned to 270 degrees
- moved SV3 97.1 mm to (96.5, 88.9), turned to 270 degrees
- moved SV5 55.7 mm to (96.5, 68.6), turned to 270 degrees
Connections:
- removed net CYCLESTART: IC9.8, LED6.A, U$2.A2
- removed net CYCLESTART_RAW: JP16.2, R15.1, R22.1
- removed net FEEDHOLD: IC9.6, LED5.A, U$2.A1
- removed net FEEDHOLD_RAW: JP15.1, R14.1, R21.1
- removed net N$10: IC1.14, U$2.D7
- removed net N$12: IC3.13, IC3.8, IC4.4, IC4.5
- removed net N$13: IC4.12, IC4.13, IC4.8, SV2.1
- removed net N$14: IC4.11, SV2.3
- removed net N$15: IC4.10, IC4.3
- removed net N$16: IC4.6, IC4.9
- removed net N$18: IC5.1, IC5.6
- removed net N$19: IC5.10, IC5.11
- removed net N$2: IC1.5, U$2.D5
- removed net N$20: IC3.10, IC3.11
- removed net N$21: IC5.3, IC5.4, IC6.1, IC6.2
- removed net N$23: IC5.13, IC5.8, IC6.4, IC6.5
- removed net N$24: IC6.11, SV3.3
- removed net N$25: IC6.10, IC6.3
- removed net N$26: IC6.6, IC6.9
- removed net N$27: IC6.12, IC6.13, IC6.8, SV3.1
- removed net N$29: IC7.1, IC7.6
- removed net N$3: IC2.3, U$2.D8
- removed net N$30: IC7.13, IC7.8
- removed net N$31: IC7.3, IC7.4, IC8.1, IC8.2
- removed net N$32: IC7.10, IC7.11, IC8.4, IC8.5
- removed net N$33: IC8.11, SV5.3
- removed net N$34: IC8.10, IC8.3
- removed net N$37: IC8.6, IC8.9
- removed net N$38: IC8.12, IC8.13, IC8.8, SV5.1
- removed net N$4: IC2.5, U$2.D13
- removed net N$40: IC2.7, U$2.D11
- removed net N$44: C2.1, IC9.1, IC9.2, R20.2
- removed net N$45: C3.1, IC9.4, IC9.5, R21.2
- removed net N$46: C4.1, IC9.10, IC9.9, R22.2
- removed net N$47: C5.1, IC9.12, IC9.13, R23.2
- removed net N$5: IC3.1, IC3.6
- removed net N$51: LED1.A, R17.2
- removed net N$53: LED2.A, R18.2
- removed net N$54: LED4.K, R24.2
- removed net N$55: LED3.A, R19.2
- removed net N$56: LED5.K, R25.2
- removed net N$57: LED6.K, R26.2
- removed net N$58: LED7.K, R27.2
- removed net N$6: IC3.3, IC3.4, IC4.1, IC4.2
- removed net N$7: IC1.7, U$2.D3
- removed net N$8: IC1.9, U$2.D6
- removed net N$9: IC1.11, U$2.D4
- removed net PROBE: IC9.11, LED7.A, U$2.A5
- removed net PROBE_RAW: JP17.3, R16.1, R23.1
- removed net RESET/ABORT: IC9.3, LED4.A, U$2.A0
- removed net RESETABORT_RAW: JP15.3, R13.1, R20.1
- removed net SPIN_DIR: IC2.4, JP7.3
- removed net SPIN_PWM: IC2.6, JP7.1
- removed net STEP_EN: IC2.2, JP2.2, JP4.2, JP6.2
- removed net STEP_X: IC1.2, JP1.3
- removed net STEP_X_DIR: IC1.4, JP1.1
- removed net STEP_Y: IC1.6, JP3.3
- removed net STEP_Y_DIR: IC1.10, JP3.1
- removed net STEP_Z: IC1.12, JP5.3
- removed net STEP_Z_DIR: IC1.15, JP5.1
- removed net X_LIM: LED1.K, SV2.2, U$2.D9
- removed net X_LIM_1_R: IC3.5, JP9.2, RN1.6
- removed net X_LIM_1_S: IC3.2, JP9.3, RN1.5
- removed net X_LIM_2_R: IC3.12, JP10.2, RN1.7
- removed net X_LIM_2_S: IC3.9, JP10.1, RN1.8
- removed net Y_LIM: LED2.K, SV3.2, U$2.D10
- removed net Y_LIM_1_R: IC5.5, JP11.2, RN1.2
- removed net Y_LIM_1_S: IC5.2, JP11.3, RN1.1
- removed net Y_LIM_2_R: IC5.12, JP12.2, RN1.3
- removed net Y_LIM_2_S: IC5.9, JP12.1, RN1.4
- removed net Z_LIM: LED3.K, SV5.2, U$2.D12
- removed net Z_LIM_1_R: IC7.5, JP13.2, RN2.6
- removed net Z_LIM_1_S: IC7.2, JP13.3, RN2.5
- removed net Z_LIM_2_R: IC7.9, JP14.2, RN2.7
- removed net Z_LIM_2_S: IC7.12, JP14.1, RN2.8
- new net B0: SV1.1, U$2.A0
- new net B1: SV2.1, U$2.A1
- new net B2: SV3.1, U$2.A2
- new net B4: SV4.1, U$2.A4
- new net B5: SV5.1, U$2.A5
- new net LIMITS0: SV6.1, U$2.D9
- new net LIMITS1: SV6.2, U$2.D10
- new net LIMITS2: SV6.3, U$2.D11
- new net SPINDLE0: SV9.1, U$2.D12
- new net SPINDLE1: SV10.1, U$2.D13
- new net STEP0: JP1.1, U$2.D2
- new net STEP1: JP3.1, U$2.D3
- new net STEP2: JP5.1, U$2.D4
- new net STEP3: JP1.3, U$2.D5
- new net STEP4: JP3.3, U$2.D6
- new net STEP5: JP5.3, U$2.D7
- new net STEP6: JP2.2, JP4.2, JP6.2, U$2.D8
- net GND: now also C1.2, JP0.3, SV1.3, SV10.3, SV11.3, SV2.3, SV3.3, SV4.3, SV5.3, SV6.4, SV9.3; no longer C2.2, C3.2, C4.2, C5.2, IC1.8, IC2.8, IC3.7, IC4.7, IC5.7, IC6.7, IC7.7, IC8.7, IC9.7, JP0.2, JP1.2, JP10.3, JP11.1, JP12.3, JP13.1, JP14.3, JP15.2, JP16.1, JP16.3, JP17.1, JP17.2, JP2.1, JP2.3, JP3.2, JP4.1, JP4.3, JP5.2, JP6.1, JP6.3, JP7.2, JP9.1, R24.1, R25.1, R26.1, R27.1
- net N$1: now also JP1.2, JP2.1, JP2.3, JP3.2, JP4.1, JP4.3, JP5.2, JP6.1, JP6.3, SV11.2; no longer IC1.3, U$2.D2
- net VCC: now also C1.1, JP0.2, SV1.2, SV10.2, SV11.1, SV2.2, SV3.2, SV4.2, SV5.2, SV9.2; no longer IC1.1, IC2.1, IC3.14, IC4.14, IC5.14, IC6.14, IC7.14, IC8.14, IC9.14, JP0.1, R13.2, R14.2, R15.2, R16.2, R17.1, R18.1, R19.1, RN1.10, RN1.11, RN1.12, RN1.13, RN1.14, RN1.15, RN1.16, RN1.9, RN2.10, RN2.11, RN2.12, RN2.9
Routing:
- net GND: track 622.7 -> 10.2 mm, vias 1 -> 4
- net PROBE: track 321.0 -> 0.00 mm, vias 9 -> 0
- net CYCLESTART: track 268.4 -> 0.00 mm, vias 6 -> 0
- net Z_LIM: track 190.6 -> 0.00 mm, vias 3 -> 0
- net RESET/ABORT: track 188.4 -> 0.00 mm, vias 2 -> 0
- net FEEDHOLD: track 173.8 -> 0.00 mm, vias 2 -> 0
- net SPINDLE1: track 0.00 -> 161.1 mm, vias 0 -> 2
- net N$1: track 42.3 -> 202.3 mm, vias 3 -> 0
- net SPINDLE0: track 0.00 -> 148.4 mm, vias 0 -> 2
- net STEP6: track 0.00 -> 145.1 mm, vias 0 -> 6
- net Y_LIM: track 139.6 -> 0.00 mm, vias 6 -> 0
- net LIMITS0: track 0.00 -> 136.7 mm
- net Y_LIM_2_R: track 126.9 -> 0.00 mm, vias 6 -> 0
- net STEP3: track 0.00 -> 126.6 mm, vias 0 -> 2
- net X_LIM_2_R: track 120.4 -> 0.00 mm, vias 7 -> 0
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- removed copper zone on layer 1, net VCC
Other:
- board size 266.7 x 48.3 mm -> 114.3 x 149.9 mm
- board text removed: "/XLIM"
- board text removed: "/YLIM"
- board text removed: "/ZLIM"
- board text removed: "1R"
- board text removed: "1S"
- board text removed: "2R"
- board text removed: "2S"
- board text removed: "CYCLE START"
- board text removed: "DIR"
- board text removed: "EN"
- board text removed: "FEED/HOLD"
- board text removed: "FEEDHOLD"
- board text removed: "GND"
- board text removed: "PROBE"
- board text removed: "PWM"
- board text removed: "RESET/ABORT"
- board text removed: "RST/ABRT"
- board text removed: "STEP"
- board text removed: "X-LIMIT"
- board text removed: "XLIM"
- board text removed: "Y-LIMIT"
- board text removed: "YLIM"
- board text removed: "Z-LIMIT"
- board text removed: "ZLIM"
