File: ArduinoMiniPro Breakout.sch (EAGLE design)
At the start: 58 parts, among them IC1 4050N, IC2 4050N, IC3 74HC00N, IC4 74HC00N, IC5 74HC00N, IC6 74HC00N, IC7 74HC00N, IC8 74HC00N, IC9 74HC00N

Commit message: Made the board a pure breakout board
Rather than smooshing all the functions onto a single board, this board
is purely for breaking out the pins to headers.

Given the relatively large size, there is no reason a full size Arduino
cannot be used, and so a full size breakout is on the way.
Parts:
- removed C2, C3, C4, C5: 10uF, SparkFun-Capacitors:CAP_POLPTH2
- removed IC1, IC2: 4050N, 40xx:4050N
- removed IC3, IC4, IC5, IC6, IC7, IC8, IC9: 74HC00N, 74xx-eu:74HC00N
- removed JP10, JP11, JP12, JP13, JP14, JP15, JP16, JP17, JP7, JP9: (no value), MY-Connectors:M03-SCREW-5MM
- removed LED1, LED2, LED3, LED4, LED5, LED6, LED7: (no value), SparkFun-LED:LED3MM
- removed R13, R14, R15, R16: 10k0, resistor:R-US_0207/7
- removed R17, R18, R19, R24, R25, R26, R27: 150, resistor:R-US_0207/7
- removed R20, R21, R22, R23: 1k00, resistor:R-US_0207/10
- removed RN1, RN2: 680, resistor-dil:8R-N
- added C1: 47uF, SparkFun-Passives:CAP_POLPTH2
- added SV1, SV11, SV4: (no value), con-lstb:MA03-1
- added SV10, SV9: (no value), SparkFun-Connectors:M03-SCREW-5MM
- added SV6: (no value), con-lstb:MA04-1
- JP1, JP2, JP3, JP4, JP5, JP6: device MY-Connectors:M03-SCREW-5MM -> SparkFun-Connectors:M03-SCREW-5MM
Connections:
- removed net CYCLESTART: IC9C.O, LED6.A, U$2.A2
- removed net CYCLESTART_RAW: JP16.2, R15.1, R22.1
- removed net FEEDHOLD: IC9B.O, LED5.A, U$2.A1
- removed net FEEDHOLD_RAW: JP15.1, R14.1, R21.1
- removed net N$10: IC1F.I, U$2.D7
- removed net N$12: IC3C.O, IC3D.I1, IC4B.I0, IC4B.I1
- removed net N$13: IC4C.O, IC4D.I0, IC4D.I1, SV2.1
- removed net N$14: IC4D.O, SV2.3
- removed net N$15: IC4A.O, IC4C.I1
- removed net N$16: IC4B.O, IC4C.I0
- removed net N$18: IC5A.I0, IC5B.O
- removed net N$19: IC5C.I1, IC5D.O
- removed net N$2: IC1B.I, U$2.D5
- removed net N$20: IC3C.I1, IC3D.O
- removed net N$21: IC5A.O, IC5B.I0, IC6A.I0, IC6A.I1
- removed net N$23: IC5C.O, IC5D.I1, IC6B.I0, IC6B.I1
- removed net N$24: IC6D.O, SV3.3
- removed net N$25: IC6A.O, IC6C.I1
- removed net N$26: IC6B.O, IC6C.I0
- removed net N$27: IC6C.O, IC6D.I0, IC6D.I1, SV3.1
- removed net N$29: IC7A.I0, IC7B.O
- removed net N$3: IC2A.I, U$2.D8
- removed net N$30: IC7C.O, IC7D.I1
- removed net N$31: IC7A.O, IC7B.I0, IC8A.I0, IC8A.I1
- removed net N$32: IC7C.I1, IC7D.O, IC8B.I0, IC8B.I1
- removed net N$33: IC8D.O, SV5.3
- removed net N$34: IC8A.O, IC8C.I1
- removed net N$37: IC8B.O, IC8C.I0
- removed net N$38: IC8C.O, IC8D.I0, IC8D.I1, SV5.1
- removed net N$4: IC2B.I, U$2.D13
- removed net N$40: IC2C.I, U$2.D11
- removed net N$44: C2.+, IC9A.I0, IC9A.I1, R20.2
- removed net N$45: C3.+, IC9B.I0, IC9B.I1, R21.2
- removed net N$46: C4.+, IC9C.I0, IC9C.I1, R22.2
- removed net N$47: C5.+, IC9D.I0, IC9D.I1, R23.2
- removed net N$5: IC3A.I0, IC3B.O
- removed net N$51: LED1.A, R17.2
- removed net N$53: LED2.A, R18.2
- removed net N$54: LED4.C, R24.2
- removed net N$55: LED3.A, R19.2
- removed net N$56: LED5.C, R25.2
- removed net N$57: LED6.C, R26.2
- removed net N$58: LED7.C, R27.2
- removed net N$6: IC3A.O, IC3B.I0, IC4A.I0, IC4A.I1
- removed net N$7: IC1C.I, U$2.D3
- removed net N$8: IC1D.I, U$2.D6
- removed net N$9: IC1E.I, U$2.D4
- removed net PROBE: IC9D.O, LED7.A, U$2.A5
- removed net PROBE_RAW: JP17.3, R16.1, R23.1
- removed net RESET/ABORT: IC9A.O, LED4.A, U$2.A0
- removed net RESETABORT_RAW: JP15.3, R13.1, R20.1
- removed net SPIN_DIR: IC2B.O, JP7.3
- removed net SPIN_PWM: IC2C.O, JP7.1
- removed net STEP_EN: IC2A.O, JP2.2, JP4.2, JP6.2
- removed net STEP_X: IC1A.O, JP1.3
- removed net STEP_X_DIR: IC1B.O, JP1.1
- removed net STEP_Y: IC1C.O, JP3.3
- removed net STEP_Y_DIR: IC1D.O, JP3.1
- removed net STEP_Z: IC1E.O, JP5.3
- removed net STEP_Z_DIR: IC1F.O, JP5.1
- removed net X_LIM: LED1.C, SV2.2, U$2.D9
- removed net X_LIM_1_R: IC3B.I1, JP9.2, RN1F.1
- removed net X_LIM_1_S: IC3A.I1, JP9.3, RN1E.1
- removed net X_LIM_2_R: IC3D.I0, JP10.2, RN1G.1
- removed net X_LIM_2_S: IC3C.I0, JP10.1, RN1H.1
- removed net Y_LIM: LED2.C, SV3.2, U$2.D10
- removed net Y_LIM_1_R: IC5B.I1, JP11.2, RN1B.1
- removed net Y_LIM_1_S: IC5A.I1, JP11.3, RN1A.1
- removed net Y_LIM_2_R: IC5D.I0, JP12.2, RN1C.1
- removed net Y_LIM_2_S: IC5C.I0, JP12.1, RN1D.1
- removed net Z_LIM: LED3.C, SV5.2, U$2.D12
- removed net Z_LIM_1_R: IC7B.I1, JP13.2, RN2F.1
- removed net Z_LIM_1_S: IC7A.I1, JP13.3, RN2E.1
- removed net Z_LIM_2_R: IC7C.I0, JP14.2, RN2G.1
- removed net Z_LIM_2_S: IC7D.I0, JP14.1, RN2H.1
- new net B0: SV1.1, U$2.A0
- new net B1: SV2.1, U$2.A1
- new net B2: SV3.1, U$2.A2
- new net B4: SV4.1, U$2.A4
- new net B5: SV5.1, U$2.A5
- new net LIMITS0: SV6.1, U$2.D9
- new net LIMITS1: SV6.2, U$2.D10
- new net LIMITS2: SV6.3, U$2.D11
- new net SPINDLE0: SV9.1, U$2.D12
- new net SPINDLE1: SV10.1, U$2.D13
- new net STEP0: JP1.1, U$2.D2
- new net STEP1: JP3.1, U$2.D3
- new net STEP2: JP5.1, U$2.D4
- new net STEP3: JP1.3, U$2.D5
- new net STEP4: JP3.3, U$2.D6
- new net STEP5: JP5.3, U$2.D7
- new net STEP6: JP2.2, JP4.2, JP6.2, U$2.D8
- net GND: now also C1.-, JP0.3, SV1.3, SV10.3, SV11.3, SV2.3, SV3.3, SV4.3, SV5.3, SV6.4, SV9.3; no longer C2.-, C3.-, C4.-, C5.-, IC1P.VSS, IC2P.VSS, IC3P.GND, IC4P.GND, IC5P.GND, IC6P.GND, IC7P.GND, IC8P.GND, IC9P.GND, JP0.2, JP1.2, JP10.3, JP11.1, JP12.3, JP13.1, JP14.3, JP15.2, JP16.1, JP16.3, JP17.1, JP17.2, JP2.1, JP2.3, JP3.2, JP4.1, JP4.3, JP5.2, JP6.1, JP6.3, JP7.2, JP9.1, R24.1, R25.1, R26.1, R27.1
- net N$1: now also JP1.2, JP2.1, JP2.3, JP3.2, JP4.1, JP4.3, JP5.2, JP6.1, JP6.3, SV11.2; no longer IC1A.I, U$2.D2
- net VCC: now also C1.+, JP0.2, SV1.2, SV10.2, SV11.1, SV2.2, SV3.2, SV4.2, SV5.2, SV9.2; no longer IC1P.VDD, IC2P.VDD, IC3P.VCC, IC4P.VCC, IC5P.VCC, IC6P.VCC, IC7P.VCC, IC8P.VCC, IC9P.VCC, JP0.1, R13.2, R14.2, R15.2, R16.2, R17.1, R18.1, R19.1, RN1A.2, RN1B.2, RN1C.2, RN1D.2, RN1E.2, RN1F.2, RN1G.2, RN1H.2, RN2E.2, RN2F.2, RN2G.2, RN2H.2
Other:
- note added: "CYCLE START/RESUME"
- note added: "DIR X"
- note added: "DIR Y"
- note added: "DIR Z"
- note added: "Debounced push button inputs"
- note added: "FEED HOLD"
- note added: "HIGH/LO SELECT"
- note added: "LIMIT X"
- note added: "LIMIT Y"
- note added: "LIMIT Z"
- note added: "PROBE"
- note added: "RESET/ABORT"
- note added: "SPINDLE DIR"
- note added: "SPINDLE ENABLE"
- note added: "STEP EN"
- note added: "STEP X"
- note added: "STEP Y"
- note added: "STEP Z"
- note added: "UNUSED"
- note removed: "Debounce"
- note removed: "MMI Debounce"
- note removed: "NOR/OR"
- note removed: "X-LIM"
- note removed: "Y-LIM"
- note removed: "Z-LIM"
- moved on the sheet: JP0, JP1, JP2, JP3, JP4, JP5, JP6, SV2, SV3, SV5
