File: Arduino Full Breakout.sch (EAGLE design)
At the start: 18 parts, among them J1 ARDUINO_R3_SHIELDUNO_R3_SHIEL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

Commit message: add pushbutton debounce to full size breakout board
Parts:
- removed JP0: (no value), MY-Connectors:M03-SCREW-5MM
- removed JP2, JP3, JP4, JP5, JP6: (no value), SparkFun-Connectors:M03-SCREW-5MM
- removed SV3, SV4, SV5: (no value), con-lstb:MA03-1
- added C2, C3, C4, C5, C6, C7: 10uF, SparkFun-Passives:CAP_POLPTH2
- added IC1, IC2: 74HC00N, 74xx-eu:74HC00N
- added R1, R11: 10k, rcl:R-EU_0207/5V
- added R10, R12, R2, R4, R6, R8: 1k00, rcl:R-EU_0207/7
- added R3, R9: 10k, rcl:R-EU_0207/7
- added R5, R7: 10k, rcl:R-EU_0207/10
- added SV12, SV13: (no value), con-lstb:MA03-1
- JP1: device SparkFun-Connectors:M03-SCREW-5MM -> con-lstb:MA03-1
- SV1: device con-lstb:MA03-1 -> SparkFun-Connectors:M03-SCREW-5MM
- SV10, SV9: device SparkFun-Connectors:M03-SCREW-5MM -> con-lstb:MA03-2
- SV11: device con-lstb:MA03-1 -> con-lstb:MA03-2
- SV2: device con-lstb:MA03-1 -> con-lstb:MA06-2
- renumbered SV6 to SV8
Connections:
- removed net B0: SV1.1
- removed net B1: SV2.1
- removed net B2: SV3.1
- removed net B4: SV4.1
- removed net B5: SV5.1
- new net BUTTONS3: IC1D.O, J1.A3
- new net N$10: C5.+, IC1D.I0, IC1D.I1, R8.1
- new net N$11: R7.1, R8.2, SV2.7
- new net N$12: C6.+, IC2C.I0, IC2C.I1, R10.1
- new net N$13: R10.2, R9.1, SV2.9
- new net N$16: C7.+, IC2D.I0, IC2D.I1, R12.1
- new net N$17: R11.1, R12.2, SV2.11
- new net N$3: C2.+, IC1B.I0, IC1B.I1, R2.1
- new net N$4: R1.1, R2.2, SV2.1
- new net N$5: C3.+, IC1A.I0, IC1A.I1, R4.1
- new net N$6: R3.1, R4.2, SV2.3
- new net N$7: C4.+, IC1C.I0, IC1C.I1, R6.1
- new net N$8: R5.1, R6.2, SV2.5
- net BUTTONS0: now also IC1B.O
- net BUTTONS1: now also IC1A.O
- net BUTTONS2: now also IC1C.O
- net BUTTONS4: now also IC2C.O
- net BUTTONS5: now also IC2D.O
- net GND: now also C2.-, C3.-, C4.-, C5.-, C6.-, C7.-, IC1P.GND, IC2A.I0, IC2A.I1, IC2B.I0, IC2B.I1, IC2P.GND, JP1.3, SV12.3, SV13.3, SV2.10, SV2.12, SV2.2, SV2.4, SV2.6, SV2.8; no longer JP0.3, SV10.3, SV11.3, SV2.3, SV3.3, SV4.3, SV5.3, SV9.3
- net N$1: now also SV10.1, SV10.3, SV10.5, SV11.1, SV11.3, SV11.5, SV9.1, SV9.3, SV9.5; no longer JP2.1, JP2.3, JP3.2, JP4.1, JP4.3, JP5.2, JP6.1, JP6.3, SV11.2
- net SPINDLE0: now also SV12.1; no longer SV9.1
- net SPINDLE1: now also SV13.1; no longer SV10.1
- net STEP0: now also SV9.6; no longer JP1.1
- net STEP1: now also SV10.6; no longer JP3.1
- net STEP2: now also SV11.6; no longer JP5.1
- net STEP3: now also SV9.4; no longer JP1.3
- net STEP4: now also SV10.4; no longer JP3.3
- net STEP5: now also SV11.4; no longer JP5.3
- net STEP6: now also SV10.2, SV11.2, SV9.2; no longer JP2.2, JP4.2, JP6.2
- net VCC: now also IC1P.VCC, IC2P.VCC, JP1.1, R1.2, R11.2, R3.2, R5.2, R7.2, R9.2, SV12.2, SV13.2; no longer JP0.2, SV10.2, SV11.1, SV2.2, SV3.2, SV4.2, SV5.2, SV9.2
Other:
- note added: "Pushbutton inputs"
- moved on the sheet: C1, JP1, SV1
